File: ESP32-C3-DevBoard.kicad_pcb (KiCad board)
At the start: 2 copper layers, 25.4 x 26 mm, 21 parts, among them J1 USB_C_Receptacle_USB2.0, J2 Conn_01x10, J3 Conn_01x10, SW1 SW_Push, SW2 SW_Push, U1 ESP32-C3-WROOM-02, U3 RT9080-33GJ5

Commit message: Add files via upload
Routing:
- net Net-(JP2-A): track 3.12 -> 3.67 mm
Changed lines of the file:
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@@
     (effects (font (size 0.8 0.8) (thickness 0.15) bold) (justify mirror))
   )
-  (gr_text "10" (at 157.48 118.745) (layer "F.SilkS")
-    (effects (font (size 0.75 0.75) (thickness 0.15) bold))
-  )
-  (gr_text "6" (at 134.62 108.585) (layer "F.SilkS")
-    (effects (font (size 0.75 0.75) (thickness 0.15) bold))
+  (gr_text "10" (at 157.48 118.7958) (layer "F.SilkS")
+    (effects (font (size 0.8 0.8) (thickness 0.15) bold))
+  )
+  (gr_text "6" (at 134.62 108.6358) (layer "F.SilkS")
+    (effects (font (size 0.8 0.8) (thickness 0.15) bold))
   )
   (gr_text "EN" (at 153.67 117.475) (layer "F.SilkS")
     (effects (font (size 0.8 0.8) (thickness 0.15) bold) (justify bottom))
   )
-  (gr_text "5V" (at 134.62 118.745) (layer "F.SilkS")
-    (effects (font (size 0.75 0.75) (thickness 0.15) bold))
+  (gr_text "5V" (at 134.62 118.7958) (layer "F.SilkS")
+    (effects (font (size 0.8 0.8) (thickness 0.15) bold))
   )
   (gr_text "BOOT" (at 138.43 117.475) (layer "F.SilkS")
     (effects (font (size 0.8 0.8) (thickness 0.15) bold) (justify bottom))
   )
-  (gr_text "2" (at 157.48 103.505) (layer "F.SilkS")
-    (effects (font (size 0.75 0.75) (thickness 0.15) bold))
-  )
-  (gr_text "TX" (at 157.48 113.665) (layer "F.SilkS")
-    (effects (font (size 0.75 0.75) (thickness 0.15) bold))
-  )
-  (gr_text "19" (at 157.48 108.585) (layer "F.SilkS")
-    (effects (font (size 0.75 0.75) (thickness 0.15) bold))
-  )
-  (gr_text "RX" (at 157.48 116.205) (layer "F.SilkS")
-    (effects (font (size 0.75 0.75) (thickness 0.15) bold))
-  )
-  (gr_text "3" (at 157.48 106.045) (layer "F.SilkS")
-    (effects (font (size 0.75 0.75) (thickness 0.15) bold))
-  )
-  (gr_text "4" (at 134.62 103.505) (layer "F.SilkS")
-    (effects (font (size 0.75 0.75) (thickness 0.15) bold))
-  )
-  (gr_text "0" (at 157.48 98.425) (layer "F.SilkS")
-    (effects (font (size 0.75 0.75) (thickness 0.15) bold))
-  )
-  (gr_text "EN" (at 134.62 100.965) (layer "F.SilkS")
-    (effects (font (size 0.75 0.75) (thickness 0.15)))
-  )
-  (gr_text "GND" (at 134.62 121.285) (layer "F.SilkS")
-    (effects (font (size 0.75 0.75) (thickness 0.15) bold))
-  )
-  (gr_text "3V3" (at 134.62 98.425) (layer "F.SilkS")
-    (effects (font (size 0.75 0.75) (thickness 0.15) bold))
-  )
-  (gr_text "1" (at 157.48 100.965) (layer "F.SilkS")
-    (effects (font (size 0.75 0.75) (thickness 0.15) bold))
-  )
-  (gr_text "9" (at 134.62 116.205) (layer "F.SilkS")
-    (effects (font (size 0.75 0.75) (thickness 0.15) bold))
-  )
-  (gr_text "8" (at 134.62 113.665) (layer "F.SilkS")
-    (effects (font (size 0.75 0.75) (thickness 0.15) bold))
-  )
-  (gr_text "18" (at 157.48 111.125) (layer "F.SilkS")
-    (effects (font (size 0.75 0.75) (thickness 0.15) bold))
+  (gr_text "2" (at 157.48 103.5558) (layer "F.SilkS")
+    (effects (font (size 0.8 0.8) (thickness 0.15) bold))
+  )
+  (gr_text "TX" (at 157.48 113.7158) (layer "F.SilkS")
+    (effects (font (size 0.8 0.8) (thickness 0.15) bold))
+  )
+  (gr_text "19" (at 157.48 108.6358) (layer "F.SilkS")
+    (effects (font (size 0.8 0.8) (thickness 0.15) bold))
+  )
+  (gr_text "RX" (at 157.48 116.2558) (layer "F.SilkS")
+    (effects (font (size 0.8 0.8) (thickness 0.15) bold))
+  )
+  (gr_text "3" (at 157.48 106.0958) (layer "F.SilkS")
+    (effects (font (size 0.8 0.8) (thickness 0.15) bold))
+  )
+  (gr_text "4" (at 134.62 103.5558) (layer "F.SilkS")
+    (effects (font (size 0.8 0.8) (thickness 0.15) bold))
+  )
+  (gr_text "0" (at 157.48 98.4758) (layer "F.SilkS")
+    (effects (font (size 0.8 0.8) (thickness 0.15) bold))
+  )
+  (gr_text "EN" (at 134.62 101.0158) (layer "F.SilkS")
+    (effects (font (size 0.8 0.8) (thickness 0.15) bold))
+  )
+  (gr_text "GND" (at 134.62 121.3358) (layer "F.SilkS")
+    (effects (font (size 0.8 0.8) (thickness 0.15) bold))
+  )
+  (gr_text "3V3" (at 134.62 98.4758) (layer "F.SilkS")
+    (effects (font (size 0.8 0.8) (thickness 0.15) bold))
+  )
+  (gr_text "1" (at 157.48 101.0158) (layer "F.SilkS")
+    (effects (font (size 0.8 0.8) (thickness 0.15) bold))
+  )
+  (gr_text "9" (at 134.62 116.2558) (layer "F.SilkS")
+    (effects (font (size 0.8 0.8) (thickness 0.15) bold))
+  )
+  (gr_text "8" (at 134.62 113.7158) (layer "F.SilkS")
+    (effects (font (size 0.8 0.8) (thickness 0.15) bold))
+  )
+  (gr_text "18" (at 157.48 111.1758) (layer "F.SilkS")
+    (effects (font (size 0.8 0.8) (thickness 0.15) bold))
   )
   (gr_text "JLCJLCJLCJLC" (at 146.05 120.015) (layer "F.SilkS")
     (effects (font (size 0.8 0.8) (thickness 0.15)))
   )
-  (gr_text "GND" (at 157.48 121.285) (layer "F.SilkS")
-    (effects (font (size 0.75 0.75) (thickness 0.15) bold))
-  )
-  (gr_text "7" (at 134.62 111.125) (layer "F.SilkS")
-    (effects (font (size 0.75 0.75) (thickness 0.15) bold))
-  )
-  (gr_text "5" (at 134.62 106.045) (layer "F.SilkS")
-    (effects (font (size 0.75 0.75) (thickness 0.15) bold))
+  (gr_text "GND" (at 157.48 121.3358) (layer "F.SilkS")
+    (effects (font (size 0.8 0.8) (thickness 0.15) bold))
+  )
+  (gr_text "7" (at 134.62 111.1758) (layer "F.SilkS")
+    (effects (font (size 0.8 0.8) (thickness 0.15) bold))
+  )
+  (gr_text "5" (at 134.62 106.0958) (layer "F.SilkS")
+    (effects (font (size 0.8 0.8) (thickness 0.15) bold))
   )
   (dimension (type aligned) (layer "Dwgs.User")
@@
   (segment (start 154.8298 98.575) (end 156.36 98.575) (width 0.25) (layer "F.Cu") (net 17))
   (segment (start 156.36 98.575) (end 157.48 99.695) (width 0.25) (layer "F.Cu") (net 17))
+  (segment (start 141.224 113.284) (end 140.8 113.284) (width 0.5) (layer "F.Cu") (net 18))
   (segment (start 141.224 113.284) (end 141.523596 113.583596) (width 0.5) (layer "F.Cu") (net 18))
-  (segment (start 141.523596 114.935) (end 141.142596 115.316) (width 0.5) (layer "F.Cu") (net 18))
-  (segment (start 140.8 113.284) (end 140.8 112.268) (width 0.5) (layer "F.Cu") (net 18))
   (segment (start 141.605 111.463) (end 141.605 101.7733) (width 0.5) (layer "F.Cu") (net 18))
   (segment (start 141.605 101.7733) (end 138.4067 98.575) (width 0.5) (layer "F.Cu") (net 18))
-  (segment (start 140.8 113.284) (end 141.224 113.284) (width 0.5) (layer "F.Cu") (net 18))
   (segment (start 141.523596 113.583596) (end 141.523596 114.935) (width 0.5) (layer "F.Cu") (net 18))
   (segment (start 137.3298 98.575) (end 135.74 98.575) (width 0.5) (layer "F.Cu") (net 18))
@@
   (segment (start 141.142596 115.316) (end 140.77 115.316) (width 0.5) (layer "F.Cu") (net 18))
   (segment (start 140.8 112.268) (end 141.605 111.463) (width 0.5) (layer "F.Cu") (net 18))
-  (via (at 140.8 113.284) (size 0.8) (drill 0.4) (layers "F.Cu" "B.Cu") (net 18))
+  (segment (start 141.523596 114.935) (end 141.142596 115.316) (width 0.5) (layer "F.Cu") (net 18))
+  (segment (start 140.8 113.284) (end 140.8 112.268) (width 0.5) (layer "F.Cu") (net 18))
+  (via (at 141.224 113.284) (size 0.8) (drill 0.4) (layers "F.Cu" "B.Cu") (net 18))
   (segment (start 147.8225 112.715) (end 149.992 112.715) (width 0.5) (layer "F.Cu") (net 19))
   (segment (start 146.311472 113.665) (end 147.261472 114.615) (width 0.5) (layer "F.Cu") (net 19))
@@
   (segment (start 139.065 115.57) (end 134.62 120.015) (width 0.5) (layer "B.Cu") (net 19))
   (segment (start 148.4 116.055) (end 148.4 116.98) (width 0.5) (layer "F.Cu") (net 20))
+  (segment (start 151.655 115.46) (end 151.231 115.884) (width 0.5) (layer "F.Cu") (net 20))
+  (segment (start 151.655 115.46) (end 152.18 114.935) (width 0.5) (layer "F.Cu") (net 20))
+  (segment (start 143.6 116.115) (end 143.6 116.98) (width 0.5) (layer "F.Cu") (net 20))
+  (segment (start 148.571 115.884) (end 148.4 116.055) (width 0.5) (layer "F.Cu") (net 20))
   (segment (start 151.231 115.884) (end 143.831 115.884) (width 0.5) (layer "F.Cu") (net 20))
-  (segment (start 148.571 115.884) (end 148.4 116.055) (width 0.5) (layer "F.Cu") (net 20))
-  (segment (start 151.9725 115.1425) (end 151.231 115.884) (width 0.5) (layer "F.Cu") (net 20))
   (segment (start 143.831 115.884) (end 143.6 116.115) (width 0.5) (layer "F.Cu") (net 20))
-  (segment (start 143.6 116.115) (end 143.6 116.98) (width 0.5) (layer "F.Cu") (net 20))
-  (via (at 151.9725 115.1425) (size 0.8) (drill 0.4) (layers "F.Cu" "B.Cu") (net 20))
-  (segment (start 151.9725 115.1425) (end 151.9725 114.6195) (width 0.5) (layer "B.Cu") (net 20))
-  (segment (start 151.9725 114.6195) (end 151.018 113.665) (width 0.5) (layer "B.Cu") (net 20))
+  (via (at 151.655 115.46) (size 0.8) (drill 0.4) (layers "F.Cu" "B.Cu") (net 20))
+  (segment (start 151.655 114.302) (end 151.018 113.665) (width 0.5) (layer "B.Cu") (net 20))
+  (segment (start 151.655 115.46) (end 151.655 114.302) (width 0.5) (layer "B.Cu") (net 20))
   (segment (start 142.621 120.015) (end 144.8 117.836) (width 0.25) (layer "F.Cu") (net 21))
   (segment (start 139.065 120.015) (end 142.621 120.015) (width 0.25) (layer "F.Cu") (net 21))
@@
   (segment (start 151.765 119.38) (end 150.945 120.2) (width 0.25) (layer "F.Cu") (net 23))
   (segment (start 144.4575 113.525) (end 145.5475 114.615) (width 0.5) (layer "F.Cu") (net 25))
-  (segment (start 142.875 113.525) (end 144.4575 113.525) (width 0.5) (layer "F.Cu") (net 25))
-  (via (at 142.875 113.525) (size 0.8) (drill 0.4) (layers "F.Cu" "B.Cu") (net 25))
+  (segment (start 142.522 113.525) (end 144.4575 113.525) (width 0.5) (layer "F.Cu") (net 25))
+  (segment (start 142.382 113.665) (end 142.522 113.525) (width 0.5) (layer "F.Cu") (net 25))
+  (via (at 142.382 113.665) (size 0.8) (drill 0.4) (layers "F.Cu" "B.Cu") (net 25))
   (zone (net 8) (net_name "GND") (layers "F&B.Cu") (hatch edge 0.5)
     (connect_pads (clearance 0.508))

Commit message: Add files via upload
Parts:
- moved SW1 15.2 mm to (153.7, 120.7)
- moved SW2 15.2 mm to (138.4, 120.7)
Routing:
- net /IO9: track 18.9 -> 37.1 mm
- net /EN: track 62.1 -> 58.3 mm
Other:
- board text added: "5V→3V3"
- board text added: "RESET"
- board text added: "VBUS=5V"
- board text removed: "DIODE"
- board text removed: "POWER"
