File: ESP32-C3-DevBoard.kicad_sch (KiCad schematic)
At the start: 19 parts, among them J1 USB_C_Receptacle_USB2.0, J2 Conn_01x10, J3 Conn_01x10, SW1 SW_Push, SW2 SW_Push, U1 ESP32-C3-WROOM-02, U2 AMS1117-3.3

Commit message: fix tooling hole position
Parts:
- U1: LCSC (none) -> C2934560; now in the parts list
Changed lines of the file:
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@@
   )
   (symbol (lib_id "PCM_Espressif:ESP32-C3-WROOM-02") (at 143.51 77.47 0) (unit 1)
-    (in_bom no) (on_board yes) (dnp no) (fields_autoplaced)
+    (in_bom yes) (on_board yes) (dnp no) (fields_autoplaced)
     (property "Reference" "U1" (at 145.4659 53.34 0)
       (effects (font (size 1.27 1.27)) (justify left))
@@
       (effects (font (size 1.27 1.27)) hide)
     )
+    (property "LCSC" "C2934560" (at 143.51 77.47 0)
+      (effects (font (size 1.27 1.27)) hide)
+    )

Commit message: Add files via upload
Parts:
- H1: value MountingHole -> ToolingHole
Changed lines of the file:
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@@
   (title_block
     (title "ESP32-C3 Development Board")
-    (rev "v1.0.0")
+    (rev "v1.0.1")
   )
   (junction (at 71.12 151.13) (diameter 0) (color 0 0 0 0)
@@
       (effects (font (size 1.27 1.27)) (justify left))
     )
-    (property "Value" "MountingHole" (at 201.93 124.46 0)
+    (property "Value" "ToolingHole" (at 201.93 124.46 0)
       (effects (font (size 1.27 1.27)) (justify left))
     )
@@
       (effects (font (size 1.27 1.27)) (justify left))
     )
-    (property "Value" "MountingHole" (at 201.93 132.08 0)
-      (effects (font (size 1.27 1.27)) (justify left))
-    )
+    (property "Value" "ToolingHole" (at 201.93 132.08 0)
+      (effects (font (size 1.27 1.27)) (justify left))
+    )

Commit message: Add Tooling Hole Library
Parts:
- H1: footprint MountingHole:MountingHole_2.2mm_M2 -> Tooling_Hole:Tooling_Hole
Changed lines of the file:
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@@
       (effects (font (size 1.27 1.27)) (justify left))
     )
-    (property "Footprint" "MountingHole:MountingHole_2.2mm_M2" (at 199.39 123.19 0)
+    (property "Footprint" "Tooling_Hole:Tooling_Hole" (at 199.39 123.19 0)
       (effects (font (size 1.27 1.27)) hide)
     )
@@
       (effects (font (size 1.27 1.27)) (justify left))
     )
-    (property "Footprint" "MountingHole:MountingHole_2.2mm_M2" (at 199.39 130.81 0)
-      (effects (font (size 1.27 1.27)) hide)
-    )
+    (property "Footprint" "Tooling_Hole:Tooling_Hole" (at 199.39 130.81 0)
+      (effects (font (size 1.27 1.27)) hide)
+    )

Commit message: Add files via upload
Parts:
- C2: value 10uF -> 22uF; LCSC C15850 -> C45783
- R1, R2: value 5.1KΩ -> 5.1kΩ
- R3, R4, R5: value 10K -> 10kΩ
Changed lines of the file:
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@@
       (effects (font (size 1.27 1.27)))
     )
-    (property "Value" "5.1KΩ" (at 83.82 66.04 90)
+    (property "Value" "5.1kΩ" (at 83.82 66.04 90)
       (effects (font (size 1 1)))
     )
@@
   (symbol (lib_id "Device:R") (at 134.62 119.38 90) (unit 1)
     (in_bom yes) (on_board yes) (dnp no) (fields_autoplaced)
-    (property "Reference" "R3" (at 134.62 114.3 90)
-      (effects (font (size 1.27 1.27)))
-    )
-    (property "Value" "10K" (at 134.62 116.84 90)
+    (property "Reference" "R3" (at 134.62 113.03 90)
+      (effects (font (size 1.27 1.27)))
+    )
+    (property "Value" "10kΩ" (at 134.62 115.57 90)
       (effects (font (size 1.27 1.27)))
     )
@@
   (symbol (lib_id "Device:R") (at 134.62 128.27 90) (unit 1)
     (in_bom yes) (on_board yes) (dnp no) (fields_autoplaced)
-    (property "Reference" "R4" (at 134.62 123.19 90)
-      (effects (font (size 1.27 1.27)))
-    )
-    (property "Value" "10K" (at 134.62 125.73 90)
+    (property "Reference" "R4" (at 134.62 121.92 90)
+      (effects (font (size 1.27 1.27)))
+    )
+    (property "Value" "10kΩ" (at 134.62 124.46 90)
       (effects (font (size 1.27 1.27)))
     )
@@
   (symbol (lib_id "Device:R") (at 134.62 138.43 90) (unit 1)
     (in_bom yes) (on_board yes) (dnp no) (fields_autoplaced)
-    (property "Reference" "R5" (at 134.62 133.35 90)
-      (effects (font (size 1.27 1.27)))
-    )
-    (property "Value" "10K" (at 134.62 135.89 90)
+    (property "Reference" "R5" (at 134.62 132.08 90)
+      (effects (font (size 1.27 1.27)))
+    )
+    (property "Value" "10kΩ" (at 134.62 134.62 90)
       (effects (font (size 1.27 1.27)))
     )
@@
       (effects (font (size 1.27 1.27)))
     )
-    (property "Value" "5.1KΩ" (at 83.82 68.58 90)
+    (property "Value" "5.1kΩ" (at 83.82 68.58 90)
       (effects (font (size 1 1)))
     )
@@
       (effects (font (size 1.27 1.27)))
     )
-    (property "Value" "10uF" (at 85.09 144.78 90)
+    (property "Value" "22uF" (at 85.09 144.78 90)
       (effects (font (size 1.27 1.27)))
     )
@@
       (effects (font (size 1.27 1.27)) hide)
     )
-    (property "Datasheet" "https://datasheet.lcsc.com/lcsc/2304140030_Samsung-Electro-Mechanics-CL21A106KAYNNNE_C15850.pdf" (at 81.28 144.78 0)
-      (effects (font (size 1.27 1.27)) hide)
-    )
-    (property "LCSC" "C15850" (at 81.28 144.78 90)
-      (effects (font (size 1.27 1.27)) hide)
-    )
+    (property "Datasheet" "https://datasheet.lcsc.com/lcsc/2304140030_Samsung-Electro-Mechanics-CL21A226MAQNNNE_C45783.pdf" (at 81.28 144.78 0)
+      (effects (font (size 1.27 1.27)) hide)
+    )
+    (property "LCSC" "C45783" (at 81.28 144.78 90)
+      (effects (font (size 1.27 1.27)) hide)
+    )

Commit message: Add files via upload
Parts:
- added JP1, JP2: Jumper_2_Open, Jumper:SolderJumper-2_P1.3mm_Open_RoundedPad1.0x1.5mm, symbol Jumper:Jumper_2_Open
- C2: footprint Capacitor_SMD:C_0805_2012Metric -> Capacitor_SMD:C_0603_1608Metric; LCSC C45783 -> C59461
Connections:
- net +3V3: now also JP2.2 (B); no longer C2.1, U2.2 (VO)
- net +5V: now also JP1.2 (B)
- net VBUS: now also JP1.1 (A)
- new net: C2.1, JP2.1 (A), U2.2 (VO)
Other:
- moved on the sheet: C1, C2, D1, U2

Commit message: Add files via upload
Parts:
- removed JP2: Jumper_2_Open, Jumper:SolderJumper-2_P1.3mm_Open_RoundedPad1.0x1.5mm, symbol Jumper:Jumper_2_Open
- removed U2: AMS1117-3.3, Package_TO_SOT_SMD:SOT-89-3, symbol Regulator_Linear:AMS1117-3.3
- added JP2: Jumper_2_Bridged, Jumper:SolderJumper-2_P1.3mm_Bridged_RoundedPad1.0x1.5mm, symbol Jumper:Jumper_2_Bridged
- added U3: RT9080-33GJ5, Package_TO_SOT_SMD:SOT-23-5, symbol Regulator_Linear:AP131-33
Connections:
- net +3V3: now also JP2.2 (B)
- net +5V: now also U3.1 (IN), U3.3 (EN)
- net GND: now also U3.2 (GND)
- net at C2.1: now also JP2.1 (A), U3.5 (OUT)
- no-connect marks 2 -> 3
Other:
- moved on the sheet: C1, C2

Commit message: Add files via upload
Parts:
- U3: LCSC C2959864 -> C841192
Changed lines of the file:
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@@
       (effects (font (size 1.27 1.27)) hide)
     )
-    (property "Datasheet" "https://datasheet.lcsc.com/lcsc/2201211530_TECH-PUBLIC-TPRT9080-33GJ5_C2959864.pdf" (at 71.12 152.4 0)
+    (property "Datasheet" "https://datasheet.lcsc.com/lcsc/2009192305_Richtek-Tech-RT9080-33GJ5_C841192.pdf" (at 71.12 152.4 0)
       (effects (font (size 1.27 1.27)) hide)
     )
-    (property "LCSC" "C2959864" (at 71.12 152.4 0)
+    (property "LCSC" "C841192" (at 71.12 152.4 0)
       (effects (font (size 1.27 1.27)) hide)
     )

Commit message: Add files via upload
Parts:
- U3: JLCPCB Rotation Offset -180 -> -90
Changed lines of the file:
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@@
       (effects (font (size 1.27 1.27)) hide)
     )
-    (property "JLCPCB Rotation Offset" "-180" (at 71.12 152.4 0)
+    (property "JLCPCB Rotation Offset" "-90" (at 71.12 152.4 0)
       (effects (font (size 1.27 1.27)) hide)
     )
