File: ESP32-C3-DevBoard.kicad_sch (KiCad schematic)
At the start: 21 parts, among them J1 USB_C_Receptacle_USB2.0_16P, J2 Conn_01x10, J3 Conn_01x10, SW1 SW_Push, SW2 SW_Push, U1 ESP32-C3-WROOM-02, U3 RT9080-33GJ5

Commit message: solder jumper fix
Parts:
- JP1: value Jumper_2_Open -> SolderJumper_2_Open; symbol Jumper:Jumper_2_Open -> Jumper:SolderJumper_2_Open
- JP2: value Jumper_2_Bridged -> SolderJumper_2_Bridged; symbol Jumper:Jumper_2_Bridged -> Jumper:SolderJumper_2_Bridged
Changed lines of the file:
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@@
+	(wire
+		(pts
+			(xy 74.93 118.11) (xy 77.47 118.11)
+		)
+		(stroke
+			(width 0)
+			(type default)
+		)
+	)
 	(wire
 		(pts
@@
 	(wire
 		(pts
-			(xy 64.77 118.11) (xy 66.04 118.11)
+			(xy 64.77 118.11) (xy 67.31 118.11)
 		)
 		(stroke
@@
 	(wire
 		(pts
-			(xy 77.47 118.11) (xy 76.2 118.11)
-		)
-		(stroke
-			(width 0)
-			(type default)
-		)
-	)
-	(wire
-		(pts
 			(xy 59.69 149.86) (xy 59.69 154.94)
 		)
@@
 	(wire
 		(pts
-			(xy 83.82 149.86) (xy 86.36 149.86)
+			(xy 83.82 149.86) (xy 87.63 149.86)
 		)
 		(stroke
@@
 	(symbol
 		(lib_id "power:+3V3")
-		(at 96.52 149.86 270)
+		(at 95.25 149.86 270)
 		(unit 1)
 		(exclude_from_sim no)
@@
 		(fields_autoplaced yes)
 		(property "Reference" "#PWR014"
-			(at 92.71 149.86 0)
+			(at 91.44 149.86 0)
 			(effects
 				(font
@@
 		)
 		(property "Value" "+3V3"
-			(at 100.33 149.86 90)
+			(at 99.06 149.86 90)
 			(effects
 				(font
@@
 		)
 		(property "Footprint" ""
-			(at 96.52 149.86 0)
+			(at 95.25 149.86 0)
 			(effects
 				(font
@@
 		)
 		(property "Datasheet" ""
-			(at 96.52 149.86 0)
+			(at 95.25 149.86 0)
 			(effects
 				(font
@@
 		)
 		(property "Description" "Power symbol creates a global label with name \"+3V3\""
-			(at 96.52 149.86 0)
+			(at 95.25 149.86 0)
 			(effects
 				(font
@@
 	)
 	(symbol
-		(lib_id "Jumper:Jumper_2_Bridged")
+		(lib_id "Jumper:SolderJumper_2_Bridged")
 		(at 91.44 149.86 0)
 		(unit 1)
-		(exclude_from_sim no)
+		(exclude_from_sim yes)
 		(in_bom no)
 		(on_board yes)
@@
 		(fields_autoplaced yes)
 		(property "Reference" "JP2"
-			(at 91.44 144.78 0)
-			(effects
-				(font
-					(size 1.27 1.27)
-				)
-			)
-		)
-		(property "Value" "Jumper_2_Bridged"
-			(at 91.44 147.32 0)
+			(at 91.44 143.51 0)
+			(effects
+				(font
+					(size 1.27 1.27)
+				)
+			)
+		)
+		(property "Value" "SolderJumper_2_Bridged"
+			(at 91.44 146.05 0)
 			(effects
 				(font
@@
 			)
 		)
-		(property "Description" "Jumper, 2-pole, closed/bridged"
+		(property "Description" "Solder Jumper, 2-pole, closed/bridged"
 			(at 91.44 149.86 0)
 			(effects
@@
 	)
 	(symbol
-		(lib_id "Jumper:Jumper_2_Open")
+		(lib_id "Jumper:SolderJumper_2_Open")
 		(at 71.12 118.11 0)
 		(unit 1)
-		(exclude_from_sim no)
+		(exclude_from_sim yes)
 		(in_bom no)
 		(on_board yes)
@@
 			)
 		)
-		(property "Value" "Jumper_2_Open"
+		(property "Value" "SolderJumper_2_Open"
 			(at 71.12 114.3 0)
 			(effects
@@
 			)
 		)
-		(property "Description" "Jumper, 2-pole, open"
+		(property "Description" "Solder Jumper, 2-pole, open"
 			(at 71.12 118.11 0)
 			(effects

Commit message: jlcpcb offset fix
Parts:
- J1: JLCPCB Position Offset 0, 1.27 -> (none)
- U3: JLCPCB Rotation Offset -90 -> 90
Changed lines of the file:
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@@
 			)
 		)
-		(property "JLCPCB Rotation Offset" "-90"
+		(property "JLCPCB Rotation Offset" "90"
 			(at 71.12 152.4 0)
 			(effects
@@
 			(at 64.77 76.2 0)
 			(effects
-				(font
-					(size 1.27 1.27)
-				)
-				(hide yes)
-			)
-		)
-		(property "JLCPCB Position Offset" "0, 1.27"
-			(at 64.77 76.2 0)
-			(effects

Commit message: change usb component
Parts:
- J1: JLCPCB Position Offset (none) -> 0, 0.13; LCSC C2765186 -> C2988369
Changed lines of the file:
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@@
 			)
 		)
-		(property "LCSC" "C2765186"
+		(property "LCSC" "C2988369"
 			(at 64.77 76.2 0)
 			(effects
+				(font
+					(size 1.27 1.27)
+				)
+				(hide yes)
+			)
+		)
+		(property "JLCPCB Position Offset" "0, 0.13"
+			(at 64.77 76.2 0)
+			(effects

Commit message: v1.1.1
Parts:
- C1: value 10uF -> 10u; LCSC C15850 -> (none); LCSC Part # (none) -> C15850
- C2: value 22uF -> 22u; LCSC C59461 -> (none); LCSC Part # (none) -> C59461
- C3: value 1uF -> 1u; LCSC C52923 -> (none); LCSC Part # (none) -> C52923
- C4: value 0.1uF -> 100n; LCSC C1525 -> (none); LCSC Part # (none) -> C1525
- D1: LCSC C191023 -> (none); LCSC Part # (none) -> C191023
- J1: FT Position Offset (none) -> 0.0, 0.13; JLCPCB Position Offset 0, 0.13 -> (none); LCSC C2988369 -> (none); LCSC Part # (none) -> C2988369
- R1, R2: value 5.1kΩ -> 5.1k
- R3, R4, R5: value 10kΩ -> 10k; LCSC C25744 -> (none); LCSC Part # (none) -> C25744
- SW1, SW2: LCSC C115360 -> (none); LCSC Part # (none) -> C115360
- U1: FT Position Offset (none) -> 0.0, -0.1; LCSC C2934560 -> (none); LCSC Part # (none) -> C2934560
- U3: FT Rotation Offset (none) -> 90; JLCPCB Rotation Offset 90 -> (none); LCSC C841192 -> (none); LCSC Part # (none) -> C841192
- renumbered H1 to H2
Other:
- moved on the sheet: C1, C2, C3, C4, D1, J1, JP1, JP2, R1, R2, R3, R4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
